File: KiCad/Luminosite/Pompe.kicad_sch (KiCad schematic)
At the start: 11 parts, among them U1 MCP6022

Commit message: Ajout des empreintes pour le PCB
Parts:
- added J1: Conn_01x03, symbol Connector_Generic:Conn_01x03
- C1, C2, C3: footprint Capacitor_SMD:C_0201_0603Metric_Pad0.64x0.40mm_HandSolder -> (none)
- D2: value BPW20RF -> D_Photo; footprint BPW20RF:TO-5_BPW20RF -> (none)
- R1, R2, R3, R4, R5, R6: footprint Resistor_SMD:R_0201_0603Metric_Pad0.64x0.40mm_HandSolder -> (none)
- U1: footprint MCP6022:SOP8P65_300X640X120L60X24N -> (none)
Connections:
- net +3.3V: now also J1.1 (Pin_1)
- net GND: now also J1.3 (Pin_3)
- net Luminosité_OUT: no longer names the net of R5.1, R6.2
- net Luminosité_OUT: now also J1.2 (Pin_2)
