File: KiCad/Luminosite/Luminosite.kicad_pcb (KiCad board)
At the start: 2 copper layers, 27 parts, among them Q1 BC547, Q2 BC547, U1 MCP6022, U2 MCP6022, U3 TL431D

Commit message: Commencement du PCB
Parts:
- removed C4: 100n, Capacitor_SMD:C_0201_0603Metric_Pad0.64x0.40mm_HandSolder
- removed Q1, Q2: BC547, Package_TO_SOT_THT:TO-92_Inline
- removed R8, R9: 10k, Resistor_SMD:R_0201_0603Metric_Pad0.64x0.40mm_HandSolder
- added C6: 100n, Capacitor_SMD:C_0603_1608Metric_Pad1.08x0.95mm_HandSolder, F.Cu at (32.7, 29.8)
- added K1: TQ2-L2-5V, TQ2-L2-5V:TQ2, F.Cu at (53.0, 57.5)
- added Q3: BC547C, BC547:TRANS_BC547C, F.Cu at (48.1, 29.1)
- added Q4: BC547C, BC547:TRANS_BC547C, F.Cu at (48.1, 40.0)
- added R16: 10k, Resistor_SMD:R_0603_1608Metric_Pad0.98x0.95mm_HandSolder, F.Cu at (37.0, 37.3)
- added R17: 10k, Resistor_SMD:R_0603_1608Metric_Pad0.98x0.95mm_HandSolder, F.Cu at (41.4, 27.3)
- added R18: 10k, Resistor_SMD:R_0603_1608Metric_Pad0.98x0.95mm_HandSolder, F.Cu at (41.4, 29.8)
- added R19: 10k, Resistor_SMD:R_0603_1608Metric_Pad0.98x0.95mm_HandSolder, F.Cu at (41.4, 32.3)
- added U4: ESP32-C3_SUPERMINI_TH, ESP32-C3-Supermini:MODULE_ESP32-C3_SUPERMINI_TH, F.Cu at (53.0, 78.0)
- C1, C2, C3, C5: footprint Capacitor_SMD:C_0201_0603Metric_Pad0.64x0.40mm_HandSolder -> Capacitor_SMD:C_0603_1608Metric_Pad1.08x0.95mm_HandSolder
- R1, R10, R11, R12, R13, R14, R15, R2, R3, R4, R5, R6, R7: footprint Resistor_SMD:R_0201_0603Metric_Pad0.64x0.40mm_HandSolder -> Resistor_SMD:R_0603_1608Metric_Pad0.98x0.95mm_HandSolder
- U1: footprint MCP6022:SOP8P65_300X640X120L60X24N -> MCP2022:SOP8P65_300X640X120L60X24N
- U2: value MCP6022 -> TL431D; footprint MCP6022:SOP8P65_300X640X120L60X24N -> Package_SO:SOIC-8_3.9x4.9mm_P1.27mm
- U3: value TL431D -> MCP6022; footprint Package_SO:SOIC-8_3.9x4.9mm_P1.27mm -> MCP2022:SOP8P65_300X640X120L60X24N
- moved U1 48.9 mm to (89.9, 75.2)
- moved D2 46.1 mm to (82.5, 43.2)
- moved R6 43.0 mm to (77.6, 83.5)
- moved R5 42.9 mm to (77.6, 81.0)
- moved R4 42.8 mm to (77.6, 78.5)
- moved R3 42.6 mm to (77.6, 76.0)
- moved R2 42.5 mm to (77.6, 73.5)
- moved R1 42.4 mm to (77.6, 71.0)
- moved C3 42.4 mm to (77.6, 68.5)
- moved C2 42.3 mm to (77.6, 66.0)
- moved C1 42.3 mm to (77.6, 63.5)
- moved U2 37.3 mm to (17.8, 37.5)
- moved C5 24.2 mm to (32.7, 27.3)
- moved R10 23.8 mm to (32.7, 34.8)
- moved R12 23.7 mm to (37.0, 27.3)
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Connections:
- R10 pad 2: Net-(U2A--) -> Net-(U3A--)
- R11 pad 1: Net-(U2A--) -> Net-(D1-K)
- R11 pad 2: Net-(R11-Pad2) -> Net-(U3A-+)
- R12 pad 1: Net-(R11-Pad2) -> GND
- R12 pad 2: Net-(U2B-+) -> Net-(U3A-+)
- R13 pad 2: Net-(U3-K) -> Net-(U2-K)
- R14 pad 1: Net-(U3-K) -> Net-(U2-K)
- R15 pad 1: VCOM -> Net-(U3A--)
- R15 pad 2: GND -> Net-(R15-Pad2)
- U2 pad 1: Net-(R11-Pad2) -> Net-(U2-K)
- U2 pad 2: Net-(U2A--) -> GND
- U2 pad 3: Net-(U2A-+) -> GND
- U2 pad 4: GND -> (no net)
- U2 pad 5: Net-(U2B-+) -> (no net)
- U2 pad 6: Net-(U2B--) -> GND
- U2 pad 7: Net-(U2B--) -> GND
- U2 pad 8: +3.3V -> Net-(U2-K)
- U3 pad 1: Net-(U3-K) -> Net-(R15-Pad2)
- U3 pad 2: GND -> Net-(U3A--)
- U3 pad 3: GND -> Net-(U3A-+)
- U3 pad 4: (no net) -> GND
- U3 pad 5: (no net) -> Net-(U3B-+)
- U3 pad 6: GND -> Net-(U3B--)
- U3 pad 7: GND -> Net-(U3B--)
- U3 pad 8: Net-(U3-K) -> +3.3V
Routing:
- net Pompe_OUT: track 0.00 -> 17.1 mm
- net unconnected-(U4-GPIO5-Pad5): track 0.00 -> 0.62 mm

Commit message: Modification du PCB
Parts:
- added J1: Conn_01x03_Pin, Connector_PinHeader_2.54mm:PinHeader_1x03_P2.54mm_Horizontal, F.Cu at (181.6, 109.2)
- moved U2 177.4 mm to (189.3, 83.2)
- moved C5 149.6 mm to (176.5, 68.5)
- moved C6 149.6 mm to (176.5, 71.0)
- moved R10 149.6 mm to (176.5, 76.1)
- moved R11 149.6 mm to (176.5, 78.6)
- moved R17 149.6 mm to (185.2, 68.5)
- moved R18 149.6 mm to (185.2, 71.0)
- moved R19 149.6 mm to (185.2, 73.5)
- moved R7 149.6 mm to (176.5, 73.5)
- moved U3 149.6 mm to (178.5, 85.7)
- moved R12 149.6 mm to (180.8, 68.5)
- moved R13 149.6 mm to (180.8, 71.0)
- moved R14 149.6 mm to (180.8, 73.5)
- moved R15 149.6 mm to (180.8, 76.1)
- moved R16 149.6 mm to (180.8, 78.6)
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Connections:
- U4 pad 21: unconnected-(U4-GPIO21-Pad21) -> Humidite_OUT
Routing:
- net Pompe_OUT: track 17.1 -> 0.00 mm
- net unconnected-(U4-GPIO5-Pad5): track 0.62 -> 0.00 mm

Commit message: Modification du PCB
Parts:
- removed D2: BPW20RF, BPW20RF:TO-5_BPW20RF
- added J2: Conn_01x02_Pin, Connector_PinHeader_2.54mm:PinHeader_1x02_P2.54mm_Horizontal, F.Cu at (121.2, 88.5)
- U4: value ESP32-C3_SUPERMINI_TH -> ESP32-C3
- moved R18 41.8 mm to (147.2, 88.5), turned to 180 degrees
- moved R19 40.7 mm to (146.3, 85.6), turned to 90 degrees
- moved Q3 39.2 mm to (157.0, 73.3), turned to -90 degrees
- moved U2 38.3 mm to (152.7, 94.2)
- moved C6 36.9 mm to (147.1, 93.5)
- moved R17 36.5 mm to (149.7, 77.0), turned to 180 degrees
- moved J1 36.1 mm to (156.6, 83.2)
- moved R13 34.1 mm to (147.0, 75.5), turned to -90 degrees
- moved R12 34.0 mm to (157.7, 93.4), turned to 90 degrees
- moved R14 33.4 mm to (147.9, 79.3)
- moved R16 33.0 mm to (149.7, 89.4), turned to -90 degrees
- moved Q4 31.6 mm to (156.3, 78.6), turned to 180 degrees
- moved C5 31.5 mm to (147.9, 81.7)
- moved R15 31.2 mm to (152.7, 89.5), turned to -90 degrees
- moved C1 31.0 mm to (123.5, 92.2), turned to -90 degrees
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Other:
- board outline added: 43.8 x 31.2 mm

Commit message: Modification du PCB
Parts:
- moved U2 10.9 mm to (156.7, 84.1)
- moved J1 7.08 mm to (156.6, 90.3)
- moved R19 6.80 mm to (148.5, 92.0), turned to 0 degrees
- moved R18 6.33 mm to (148.5, 94.7)
- moved R12 5.88 mm to (152.8, 96.8)
- moved U1 5.79 mm to (136.2, 96.8)
- moved C6 4.14 mm to (148.5, 97.4)
- moved R15 3.38 mm to (152.8, 92.8)
- moved R16 3.19 mm to (152.8, 88.9)
- moved U3 2.05 mm to (149.3, 86.8), turned to -90 degrees
- moved R2 0.77 mm to (124.4, 97.3)
- moved C3 0.70 mm to (124.4, 95.4)
- moved C2 0.33 mm to (119.9, 97.3)
- moved R4 0.33 mm to (119.9, 95.4)
- moved C1 0.25 mm to (123.5, 92.5)
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Other:
- board size 43.8 x 31.2 mm -> 43.8 x 29.6 mm

Commit message: Modification du PCB
Parts:
- added J3: Conn_01x02_Pin, Connector_PinHeader_2.54mm:PinHeader_1x02_P2.54mm_Horizontal, F.Cu at (121.2, 88.6)
- U4: value ESP32-C3 -> ESP32-C3_SUPERMINI_TH
- moved C2 12.0 mm to (132.0, 97.4), turned to 180 degrees
- moved R4 12.0 mm to (131.9, 95.5)
- moved C3 11.4 mm to (135.8, 95.5)
- moved R2 11.4 mm to (135.8, 97.3)
- moved R3 10.0 mm to (128.3, 96.4)
- moved J2 7.73 mm to (121.2, 96.2)
- moved R1 6.75 mm to (126.2, 96.4), turned to 90 degrees
- moved U1 6.20 mm to (142.4, 96.6)
- moved C1 4.03 mm to (124.2, 96.4), turned to 90 degrees
- moved R6 1.68 mm to (125.1, 91.4)
- moved R5 1.68 mm to (125.1, 87.5)
- turned K1 to 90 degrees
Connections:
- K1 pad 4: Alim Pompe -> Net-(J3-Pin_2)
Routing:
- net Pompe_OUT: track 0.00 -> 7.68 mm

Commit message: Modification du PCB
Parts:
- moved C6 25.5 mm to (156.7, 73.2), turned to 90 degrees
- moved R12 24.2 mm to (158.6, 73.2), turned to -90 degrees
- moved J1 20.6 mm to (147.0, 72.0), turned to 90 degrees
- moved R17 15.5 mm to (151.1, 92.4)
- moved R15 14.0 mm to (151.2, 79.0), turned to 180 degrees
- moved R16 11.3 mm to (147.6, 79.0), turned to 180 degrees
- moved R14 11.1 mm to (151.1, 90.0), turned to 180 degrees
- moved R13 10.8 mm to (147.2, 86.3)
- moved R7 10.1 mm to (151.1, 84.6)
- moved Q3 6.81 mm to (156.8, 80.1), turned to 0 degrees
- moved C5 6.76 mm to (152.0, 87.1), turned to 90 degrees
- moved R10 6.65 mm to (150.3, 87.1), turned to 90 degrees
- moved U2 6.18 mm to (156.8, 90.3)
- moved D1 4.83 mm to (154.3, 76.0)
- moved Q4 4.83 mm to (156.8, 83.4)
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Connections:
- J1 pad 2: GND_ESP32 -> GND
- U4 pad 21: Humidite_OUT -> unconnected-(U4-GPIO21-Pad21)
- U4 pad 5: unconnected-(U4-GPIO5-Pad5) -> Humidite_OUT
- U4 pad G: GND_ESP32 -> GND
Routing:
- net Humidite_OUT: track 0.00 -> 25.3 mm
- net Net-(U3B-+): track 0.00 -> 18.2 mm
- net Net-(U2-K): track 0.00 -> 15.0 mm
- net GND: track 0.00 -> 13.6 mm
- net +3.3V: track 0.00 -> 13.1 mm
- net Net-(U3A-+): track 0.00 -> 11.9 mm
- net Net-(Q3-Pad2): track 0.00 -> 11.1 mm
- net Net-(U3A--): track 0.00 -> 10.8 mm
- net Net-(R15-Pad2): track 0.00 -> 6.91 mm
- net Net-(D1-K): track 0.00 -> 6.57 mm
- net VCOM: track 0.00 -> 6.19 mm
- net +5V: track 0.00 -> 3.78 mm
- net Net-(U3B--): track 0.00 -> 3.12 mm
- net Température_OUT: track 0.00 -> 2.41 mm

Commit message: PCB Terminé
Parts:
- added J4: Conn_01x02_Pin, Connector_PinHeader_2.54mm:PinHeader_1x02_P2.54mm_Horizontal, F.Cu at (123.3, 73.5)
- added U5: AMS1117-5.0, Package_TO_SOT_SMD:SOT-223-3_TabPin2, F.Cu at (122.8, 87.8)
- moved C1 27.2 mm to (151.0, 100.3)
- moved R3 27.0 mm to (155.0, 100.3)
- moved R1 26.8 mm to (152.7, 100.3)
- moved R4 26.6 mm to (158.5, 97.8)
- moved C2 24.0 mm to (155.9, 96.9), turned to 90 degrees
- moved C3 23.0 mm to (158.5, 99.5), turned to 0 degrees
- moved K1 21.7 mm to (126.2, 98.2), turned to 180 degrees
- moved R5 21.1 mm to (143.9, 97.2), turned to 0 degrees
- moved R6 20.2 mm to (143.9, 98.9), turned to 180 degrees
- moved J2 17.6 mm to (138.6, 99.1), turned to -90 degrees
- moved R2 17.5 mm to (153.3, 97.8), turned to 0 degrees
- moved J3 8.12 mm to (123.3, 80.7)
- moved U1 7.48 mm to (148.0, 98.2), turned to 90 degrees
- moved R19 5.45 mm to (147.1, 84.6)
- moved R18 5.45 mm to (147.1, 87.0)
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Connections:
- J3 pad 1: GND -> Net-(J3-Pin_1)
- K1 pad 3: +5V -> Net-(U5-VO)
- U4 pad 10: Luminosité_OUT -> unconnected-(U4-GPIO10-Pad10)
- U4 pad 20: unconnected-(U4-GPIO20-Pad20) -> Pompe_OUT
- U4 pad 21: unconnected-(U4-GPIO21-Pad21) -> Luminosité_OUT
- U4 pad 4: unconnected-(U4-GPIO4-Pad4) -> Humidite_OUT
- U4 pad 5: Humidite_OUT -> unconnected-(U4-GPIO5-Pad5)
- U4 pad 6: Pompe_OUT -> unconnected-(U4-GPIO6-Pad6)
Routing:
- net Luminosité_OUT: track 0.00 -> 19.9 mm
- net Net-(J3-Pin_2): track 0.00 -> 18.8 mm
- net Net-(J2-Pin_1): track 0.00 -> 17.3 mm
- net +3.3V: track 13.1 -> 29.9 mm
- net Net-(J3-Pin_1): track 0.00 -> 15.4 mm
- net Net-(U1B-+): track 0.00 -> 14.5 mm
- net Net-(U1A-+): track 0.00 -> 14.2 mm
- net Net-(U1B--): track 0.00 -> 13.3 mm
- net Net-(J4-Pin_1): track 0.00 -> 12.3 mm
- net GND: track 13.6 -> 25.1 mm, vias 0 -> 9
- net Net-(U5-VO): track 0.00 -> 11.1 mm
- net Humidite_OUT: track 25.3 -> 15.2 mm
- net Net-(C1-Pad2): track 0.00 -> 9.17 mm
- net Net-(C2-Pad1): track 0.00 -> 6.28 mm
- net Température_OUT: track 2.41 -> 6.10 mm
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- added copper zone on B.Cu, net GND
Other:
- board size 43.8 x 29.6 mm -> 42 x 34.8 mm

Commit message: Doc Commande
Parts:
- U4: value ESP32-C3_SUPERMINI_TH -> ESP32-C3_SUPERMINI
- moved K1 0.42 mm to (126.5, 98.5)
- moved J2 0.20 mm to (138.6, 99.3)
Other:
- board size 42 x 34.8 mm -> 42 x 35 mm
- board text added: "Batterie"
- board text added: "Humidité"
- board text added: "Luminosité"
- board text added: "Pompe"
Changed lines of the file:
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@@
 		(tags "Through hole angled pin header THT 1x02 2.54mm single row")
 		(property "Reference" "J4"
-			(at -1.3 -2.4 0)
+			(at -1.49 -2.2 0)
 			(layer "F.SilkS")
 			(effects
@@
 		(tags "Through hole angled pin header THT 1x03 2.54mm single row")
 		(property "Reference" "J1"
-			(at 3.535 7.39 180)
+			(at 2.235 7.315 180)
 			(layer "F.SilkS")
 			(effects
@@
 	(footprint "Connector_PinHeader_2.54mm:PinHeader_1x02_P2.54mm_Horizontal"
 		(layer "F.Cu")
-		(at 138.6 99.14 -90)
+		(at 138.6 99.34 -90)
 		(descr "Through hole angled pin header, 1x02, 2.54mm pitch, 6mm pin length, single row")
 		(tags "Through hole angled pin header THT 1x02 2.54mm single row")
@@
 			)
 		)
-		(property "Value" "ESP32-C3_SUPERMINI_TH"
-			(at -0.275 -11.95 180)
+		(property "Value" "ESP32-C3_SUPERMINI"
+			(at 0 -11.825 180)
 			(layer "F.Fab")
 			(effects
@@
 	(footprint "TQ2-L2-5V:TQ2"
 		(layer "F.Cu")
-		(at 126.175 98.2 180)
+		(at 126.475 98.5 180)
 		(descr "2 Form C (DPDT-BM) / Dimensions L x W x H 14 x 9 x 5mm")
 		(property "Reference" "K1"
@@
 	(gr_rect
 		(start 119.049999 68.6)
-		(end 161.05 103.375)
+		(end 161.05 103.6)
 		(stroke
 			(width 0.05)
@@
 		(layer "Edge.Cuts")
 	)
+	(gr_text "Luminosité"
+		(at 134.2 97.275 0)
+		(layer "F.Cu")
+		(effects
+			(font
+				(size 0.8 0.8)
+				(thickness 0.15)
+			)
+			(justify left bottom)
+		)
+	)
+	(gr_text "Humidité"
+		(at 153.925 70.15 0)
+		(layer "F.Cu")
+		(effects
+			(font
+				(size 0.8 0.8)
+				(thickness 0.15)
+			)
+			(justify left bottom)
+		)
+	)
+	(gr_text "Batterie"
+		(at 125.35 70.15 270)
+		(layer "F.Cu")
+		(effects
+			(font
+				(size 0.8 0.8)
+				(thickness 0.15)
+			)
+			(justify left bottom)
+		)
+	)
+	(gr_text "Pompe"
+		(at 125.4 77.35 270)
+		(layer "F.Cu")
+		(effects
+			(font
+				(size 0.8 0.8)
+				(thickness 0.15)
+			)
+			(justify left bottom)
+		)
+	)
 	(segment
 		(start 149.1725 101.25)
@@
 	)
 	(segment
-		(start 123.635 94.39)
-		(end 123.201358 94.39)
+		(start 120.65 91.838642)
+		(end 123.501358 94.69)
 		(width 0.2)
 		(layer "F.Cu")
@@
 	)
 	(segment
-		(start 121.8 85.604594)
-		(end 121.8 79.695)
+		(start 123.501358 94.69)
+		(end 123.935 94.69)
 		(width 0.2)
 		(layer "F.Cu")
@@
 	)
 	(segment
-		(start 123.201358 94.39)
-		(end 120.65 91.838642)
+		(start 121.8 85.604594)
+		(end 121.8 79.695)
 		(width 0.2)
 		(layer "F.Cu")
@@
 	)
 	(segment
-		(start 138.865 99.14)
-		(end 141.695 101.97)
+		(start 151.0475 101.2)
+		(end 149.9275 100.08)
 		(width 0.2)
 		(layer "F.Cu")
@@
 	)
 	(segment
-		(start 151.0475 101.2)
-		(end 149.9275 100.08)
+		(start 147.6475 100.468414)
+		(end 147.6475 101.025)
 		(width 0.2)
 		(layer "F.Cu")
@@
 	)
 	(segment
-		(start 147.6475 100.468414)
-		(end 147.6475 101.025)
+		(start 139.065 99.34)
+		(end 138.6 99.34)
 		(width 0.2)
 		(layer "F.Cu")
@@
 	)
 	(segment
+		(start 141.695 101.97)
+		(end 139.065 99.34)
+		(width 0.2)
+		(layer "F.Cu")
+		(net "Net-(J2-Pin_1)")
+	)
+	(segment
 		(start 152.7225 101.275)
 		(end 151.1225 101.275)
@@
 	)
 	(segment
-		(start 122.85 91.065)
-		(end 122.85 91)
+		(start 126.475 94.625)
+		(end 126.475 94.69)
 		(width 0.2)
 		(layer "F.Cu")
@@
 	)
 	(segment
-		(start 126.175 94.39)
-		(end 122.85 91.065)
+		(start 122.85 91)
+		(end 126.475 94.625)
 		(width 0.2)
 		(layer "F.Cu")
@@
 	)
 	(segment
+		(start 122.85 91.065)
+		(end 122.85 91)
+		(width 0.2)
+		(layer "F.Cu")
+		(net "Net-(U5-VO)")
+	)
+	(segment
 		(start 148.725 88.335778)
 		(end 148.725 89.75)
@@
 	(segment
 		(start 127.125 90.26)
-		(end 127.125 88.295)
+		(end 131.555 94.69)
 		(width 0.2)
 		(layer "F.Cu")
@@
 	)
 	(segment
-		(start 131.255 94.39)
-		(end 127.125 90.26)
+		(start 127.125 90.26)
+		(end 127.125 88.295)
 		(width 0.2)
 		(layer "F.Cu")
@@
 		(polygon
 			(pts
-				(xy 116.75 68.325) (xy 161.225 68.325) (xy 161.225 103.825) (xy 116.723922 103.825) (xy 116.775 68.275)
+				(xy 116.75 68.325) (xy 161.225 68.325) (xy 161.225 103.825) (xy 118.646694 103.825) (xy 118.703313 64.418374)
 			)
 		)
