File: KiCad/Luminosite/Luminosite.kicad_pcb (KiCad board)
At the start: 2 copper layers, 42 x 35 mm, 35 parts, among them J1 Conn_01x03_Pin, J2 Conn_01x02_Pin, J3 Conn_01x02_Pin, J4 Conn_01x02_Pin, K1 TQ2-L2-5V, Q3 BC547C, Q4 BC547C, U1 MCP6022, U2 TL431D, U3 MCP6022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

Commit message: Finalisation PCB
Routing:
- net Net-(J3-Pin_2): track 19.2 -> 20.9 mm
- net Net-(J3-Pin_1): track 15.4 -> 17.2 mm
- net Pompe_OUT: track 9.90 -> 10.5 mm
- net GND: track 25.1 -> 24.6 mm
Changed lines of the file:
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@@
 		(layer "Edge.Cuts")
+	)
+	(gr_text "Humidité"
+		(at 154 70.225 0)
+		(layer "F.Cu")
+		(effects
+			(font
+				(size 0.7 0.7)
+				(thickness 0.15)
+			)
+			(justify left bottom)
+		)
+	)
+	(gr_text "Pompe"
+		(at 125.7 77.85 270)
+		(layer "F.Cu")
+		(effects
+			(font
+				(size 0.7 0.7)
+				(thickness 0.15)
+			)
+			(justify left bottom)
+		)
+	)
+	(gr_text "Batterie"
+		(at 125.725 70.35 270)
+		(layer "F.Cu")
+		(effects
+			(font
+				(size 0.7 0.7)
+				(thickness 0.15)
+			)
+			(justify left bottom)
+		)
 	)
 	(gr_text "Luminosité"
@@
 		)
 	)
-	(gr_text "Humidité"
-		(at 153.925 70.15 0)
-		(layer "F.Cu")
-		(effects
-			(font
-				(size 0.8 0.8)
-				(thickness 0.15)
-			)
-			(justify left bottom)
-		)
-	)
-	(gr_text "Batterie"
-		(at 125.35 70.15 270)
-		(layer "F.Cu")
-		(effects
-			(font
-				(size 0.8 0.8)
-				(thickness 0.15)
-			)
-			(justify left bottom)
-		)
-	)
-	(gr_text "Pompe"
-		(at 125.4 77.35 270)
-		(layer "F.Cu")
-		(effects
-			(font
-				(size 0.8 0.8)
-				(thickness 0.15)
-			)
-			(justify left bottom)
-		)
-	)
 	(segment
 		(start 149.1725 101.25)
@@
 	)
 	(segment
+		(start 156.735 70.95)
+		(end 156.735 72.325)
+		(width 0.2)
+		(layer "F.Cu")
+		(net "GND")
+	)
+	(segment
 		(start 152.445 86.28)
 		(end 153.125 85.6)
@@
 	)
 	(segment
-		(start 156.735 70.465)
-		(end 156.75 70.45)
-		(width 0.2)
-		(layer "F.Cu")
-		(net "GND")
-	)
-	(segment
 		(start 154.25 96.65)
 		(end 154.25 96.775)
@@
 		(start 144.7725 100.4975)
 		(end 144.775 100.5)
-		(width 0.2)
-		(layer "F.Cu")
-		(net "GND")
-	)
-	(segment
-		(start 156.735 72.325)
-		(end 156.735 70.465)
 		(width 0.2)
 		(layer "F.Cu")
@@
 	)
 	(via
-		(at 156.75 70.45)
+		(at 156.735 70.95)
 		(size 0.6)
 		(drill 0.3)
@@
 	)
 	(segment
-		(start 124.485 72.135)
-		(end 124.485 79.55)
+		(start 123.31 80.725)
+		(end 123.31 82.235)
 		(width 0.2)
 		(layer "F.Cu")
@@
 	)
 	(segment
-		(start 123.31 80.725)
-		(end 123.31 82.86)
+		(start 125.15 84.075)
+		(end 125.15 84.7)
 		(width 0.2)
 		(layer "F.Cu")
@@
 	)
 	(segment
-		(start 124.485 79.55)
+		(start 125.325 79.459038)
+		(end 124.059038 80.725)
+		(width 0.2)
+		(layer "F.Cu")
+		(net "Net-(J3-Pin_1)")
+	)
+	(segment
+		(start 123.335 70.985)
+		(end 124.335 70.985)
+		(width 0.2)
+		(layer "F.Cu")
+		(net "Net-(J3-Pin_1)")
+	)
+	(segment
+		(start 125.325 71.975)
+		(end 125.325 79.459038)
+		(width 0.2)
+		(layer "F.Cu")
+		(net "Net-(J3-Pin_1)")
+	)
+	(segment
+		(start 124.335 70.985)
+		(end 125.325 71.975)
+		(width 0.2)
+		(layer "F.Cu")
+		(net "Net-(J3-Pin_1)")
+	)
+	(segment
+		(start 124.059038 80.725)
 		(end 123.31 80.725)
 		(width 0.2)
@@
 	)
 	(segment
-		(start 123.335 70.985)
-		(end 124.485 72.135)
+		(start 123.31 82.235)
+		(end 125.15 84.075)
 		(width 0.2)
 		(layer "F.Cu")
@@
 	)
 	(segment
-		(start 123.31 82.86)
-		(end 125.15 84.7)
-		(width 0.2)
-		(layer "F.Cu")
-		(net "Net-(J3-Pin_1)")
-	)
-	(segment
-		(start 120.65 91.838642)
-		(end 120.65 86.754594)
+		(start 120.25 91.7)
+		(end 123.24 94.69)
 		(width 0.2)
 		(layer "F.Cu")
@@
 	)
 	(segment
-		(start 120.65 86.754594)
-		(end 121.8 85.604594)
+		(start 120.25 87.725)
+		(end 120.25 91.7)
 		(width 0.2)
 		(layer "F.Cu")
@@
 	)
 	(segment
-		(start 120.65 91.838642)
-		(end 123.501358 94.69)
+		(start 123.24 94.69)
+		(end 123.935 94.69)
 		(width 0.2)
 		(layer "F.Cu")
@@
 	)
 	(segment
-		(start 123.501358 94.69)
-		(end 123.935 94.69)
+		(start 121.175 79)
+		(end 121.15 79)
 		(width 0.2)
 		(layer "F.Cu")
@@
 	)
 	(segment
-		(start 121.8 85.604594)
-		(end 121.8 79.695)
+		(start 121.7 83.375)
+		(end 121.7 86.275)
 		(width 0.2)
 		(layer "F.Cu")
@@
 	)
 	(segment
-		(start 121.8 79.695)
-		(end 123.31 78.185)
+		(start 121.7 86.275)
+		(end 120.25 87.725)
+		(width 0.2)
+		(layer "F.Cu")
+		(net "Net-(J3-Pin_2)")
+	)
+	(segment
+		(start 123.31 78.185)
+		(end 121.99 78.185)
+		(width 0.2)
+		(layer "F.Cu")
+		(net "Net-(J3-Pin_2)")
+	)
+	(segment
+		(start 121.15 79)
+		(end 121.15 82.825)
+		(width 0.2)
+		(layer "F.Cu")
+		(net "Net-(J3-Pin_2)")
+	)
+	(segment
+		(start 121.99 78.185)
+		(end 121.175 79)
+		(width 0.2)
+		(layer "F.Cu")
+		(net "Net-(J3-Pin_2)")
+	)
+	(segment
+		(start 121.15 82.825)
+		(end 121.7 83.375)
 		(width 0.2)
 		(layer "F.Cu")
@@
 	)
 	(segment
-		(start 127.125 90.26)
-		(end 131.555 94.69)
+		(start 131.555 94.69)
+		(end 130.965 94.69)
 		(width 0.2)
 		(layer "F.Cu")
@@
 	)
 	(segment
-		(start 127.125 90.26)
-		(end 127.125 88.295)
+		(start 126.8 88.62)
+		(end 128.305 87.115)
 		(width 0.2)
 		(layer "F.Cu")
@@
 	)
 	(segment
-		(start 127.125 88.295)
-		(end 128.305 87.115)
+		(start 130.965 94.69)
+		(end 126.8 90.525)
+		(width 0.2)
+		(layer "F.Cu")
+		(net "Pompe_OUT")
+	)
+	(segment
+		(start 126.8 90.525)
+		(end 126.8 88.62)
 		(width 0.2)
 		(layer "F.Cu")
@@
 		(polygon
 			(pts
-				(xy 116.75 68.325) (xy 161.225 68.325) (xy 161.225 103.825) (xy 118.646694 103.825) (xy 118.703313 64.418374)
+				(xy 118.704765 68.34074) (xy 161.225 68.325) (xy 161.225 103.825) (xy 118.646694 103.825) (xy 118.721368 68.357413)
 			)
 		)

Commit message: Maj
Parts:
- added C4: 10p, Capacitor_SMD:C_0603_1608Metric_Pad1.08x0.95mm_HandSolder, F.Cu at (143.5, 99.6)
- U4: value ESP32-C3_SUPERMINI -> ESP32-C3_SUPERMINI_TH
- moved R5 1.15 mm to (143.5, 96.1)
- moved R6 1.15 mm to (143.5, 97.8)
Routing:
- net Luminosité_OUT: track 19.9 -> 22.0 mm
- net GND: track 24.6 -> 26.4 mm
- net Net-(U1B--): track 13.3 -> 14.1 mm

Commit message: Maj
Changed lines of the file:
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@@
 			(outputformat 1)
 			(mirror no)
-			(drillshape 1)
+			(drillshape 0)
 			(scaleselection 1)
-			(outputdirectory "")
+			(outputdirectory "Gerber/")
 		)
 	)
@@
 		(at 147.9725 98.205 90)
 		(property "Reference" "U1"
-			(at 3.2 -2.15 90)
+			(at -0.345 -2.1225 90)
 			(layer "F.SilkS")
 			(effects
@@
 		(tags "CMS SOT")
 		(property "Reference" "U5"
-			(at 4.925 3.25 180)
+			(at 4.9 3.075 180)
 			(layer "F.SilkS")
 			(effects
@@
 		)
 		(property "Value" "ESP32-C3_SUPERMINI_TH"
-			(at 0 -11.825 180)
+			(at -0.025 -10.675 180)
 			(layer "F.Fab")
 			(effects
@@
 	(gr_text "Humidité"
 		(at 154 70.225 0)
-		(layer "F.Cu")
+		(layer "F.SilkS")
 		(effects
 			(font
@@
 	(gr_text "Pompe"
 		(at 125.7 77.85 270)
-		(layer "F.Cu")
+		(layer "F.SilkS")
 		(effects
 			(font
@@
 	(gr_text "Batterie"
 		(at 125.725 70.35 270)
-		(layer "F.Cu")
+		(layer "F.SilkS")
 		(effects
 			(font
@@
 	(gr_text "Luminosité"
 		(at 134.2 97.275 0)
-		(layer "F.Cu")
+		(layer "F.SilkS")
 		(effects
 			(font
